Commit message: PHASE 3: SLAM 준비 — URDF laser 프레임 정리 + slam_toolbox 설정/launch 추가
- URDF: lidar_link → laser 프레임 통일 (rplidar /scan frame_id 와 일치)
- URDF: odom 링크 제거 (odom→base_link 은 base_controller 가 동적 발행)
- config/slam_toolbox.yaml: base_frame=base_link, max_laser_range=12.0 (A1M8)
- launch/slam.launch.py: 데스크탑용 SLAM 한 줄 실행
- setup.py: config/ 설치 등록
- NOTES.md, .feature/skills/lint 추가

File: ros2_ws/src/autonomous_robot/urdf/robot.urdf (robot description, URDF)
Before this commit: robot autonomous_robot, 7 links, 6 joints
Links:
- removed link lidar_link
- removed link odom
- added link laser
Joints:
- removed joint lidar_joint
- removed joint odom_base_joint
- added joint laser_joint: type fixed, parent base_link, child laser, origin xyz=0 0 0.10 rpy=0 0 0
